File: drivers/Hoperf Electronic/RFM70/doc/hardware/breakout board/eagle/rfm70.sch (EAGLE design)
At the start: 4 parts, among them CON1 MICROHAL_CONNECTOR_M_1_REDUCE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

Commit message: RFM70 PCB - fixed bug on PCB.
Connections:
- net MISO: now also CON1.MISO; no longer CON1.MOSI
- net MOSI: now also CON1.MOSI; no longer CON1.MISO
Changed lines of the file:
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@@
 <?xml version="1.0" encoding="utf-8"?>
 <!DOCTYPE eagle SYSTEM "eagle.dtd">
-<eagle version="7.3.0">
+<eagle version="7.5.0">
 <drawing>
 <settings>
@@
 <net name="MOSI" class="0">
 <segment>
-<pinref part="CON1" gate="G$1" pin="MISO"/>
-<wire x1="76.2" y1="142.24" x2="66.04" y2="142.24" width="0.1524" layer="91"/>
-<label x="66.04" y="142.24" size="1.27" layer="95" rot="R180" xref="yes"/>
+<label x="66.04" y="139.7" size="1.27" layer="95" rot="R180" xref="yes"/>
+<pinref part="CON1" gate="G$1" pin="MOSI"/>
+<wire x1="66.04" y1="139.7" x2="76.2" y2="139.7" width="0.1524" layer="91"/>
 </segment>
 <segment>
@@
 <net name="MISO" class="0">
 <segment>
-<pinref part="CON1" gate="G$1" pin="MOSI"/>
-<wire x1="76.2" y1="139.7" x2="66.04" y2="139.7" width="0.1524" layer="91"/>
-<label x="66.04" y="139.7" size="1.27" layer="95" rot="R180" xref="yes"/>
+<label x="66.04" y="142.24" size="1.27" layer="95" rot="R180" xref="yes"/>
+<pinref part="CON1" gate="G$1" pin="MISO"/>
+<wire x1="66.04" y1="142.24" x2="76.2" y2="142.24" width="0.1524" layer="91"/>
 </segment>
 <segment>
